File: KiCad Circuit/SolarCarSchematic.kicad_sch (KiCad schematic)
At the start: 21 parts, among them Q1 BS250, Q2 NMOS, Q3 IPP060N06N, Q4 PMOS, U1 TL494

Commit message: KiCad schematic with updated accurate values
Parts:
- removed Q4: PMOS, symbol Simulation_SPICE:PMOS
- added C6: 220u, symbol Device:C
- added C7: 100n, symbol Device:C
- C3: value 2.2u? -> 47u
- C4: value 100n -> 1u
- MOTOR_LOAD: renamed from R8; value R -> 3
- Q2: value NMOS -> BS270
- R4: value 100 -> 1k
- R5: value 10 -> 100
- R7: value 100k -> 1M
- renumbered RV1 to POTENTIOMETER
Connections:
- net GND: now also C6.2, C7.2
- net VCC: now also C6.1, C7.1
Other:
- title: (none) -> Solar Car Schematic
